File: hardware/v1/v1.kicad_sch (KiCad schematic)
At the start: 1 part

Commit message: Schem and PCB
Parts:
- added C1: 100u, Capacitor_THT:CP_Radial_D7.5mm_P2.50mm, symbol Device:C_Polarized
- added C2, C4: 100n, Capacitor_THT:C_Axial_L3.8mm_D2.6mm_P7.50mm_Horizontal, symbol Device:C
- added C3: 1000u, Capacitor_THT:CP_Radial_D10.0mm_P5.00mm, symbol Device:C_Polarized
- added D1: 1N914, Diode_THT:D_DO-34_SOD68_P7.62mm_Horizontal, symbol Device:D
- added H1, H2, H3, H4, H5, H6, H7, H8: MountingHole, MountingHole:MountingHole_3.2mm_M3, symbol Mechanical:MountingHole
- added J1: MIDI in TRS, MIDI_TRS:PJ-320B, symbol Connector:AudioJack3
- added J10: Batt, Connector_JST:JST_XH_B2B-XH-A_1x02_P2.50mm_Vertical, symbol Connector:Conn_01x02_Female
- added J2: MIDI IN, MIDI_DIN5:DS-5 MIDI_Wide, symbol Connector:DIN-5_180degree
- added J3: MIDI THRU, MIDI_DIN5:DS-5 MIDI_Wide, symbol Connector:DIN-5_180degree
- added J4: MIDI thru TRS, MIDI_TRS:PJ-320B, symbol Connector:AudioJack3
- added J5: SSD1306 - I2C, Connector_JST:JST_EH_B4B-EH-A_1x04_P2.50mm_Vertical, symbol Connector:Conn_01x04_Female
- added J6: DotStar1/k:GND, Connector_JST:JST_PH_S4B-PH-K_1x04_P2.00mm_Horizontal, symbol Connector:Conn_01x04_Female
- added J7: DotStar2/k:GND, Connector_JST:JST_PH_S4B-PH-K_1x04_P2.00mm_Horizontal, symbol Connector:Conn_01x04_Female
- added J8: Barrel_Jack_Switch, Connector_BarrelJack:BarrelJack_CUI_PJ-102AH_Horizontal, symbol Connector:Barrel_Jack_Switch
- added J9: On/Off, Connector_JST:JST_XH_B2B-XH-A_1x02_P2.50mm_Vertical, symbol Connector:Conn_01x02_Female
- added R1, R2: 220, Resistor_THT:R_Axial_DIN0207_L6.3mm_D2.5mm_P7.62mm_Horizontal, symbol Device:R
- added R3: 33, Resistor_THT:R_Axial_DIN0207_L6.3mm_D2.5mm_P7.62mm_Horizontal, symbol Device:R
- added R4: 10, Resistor_THT:R_Axial_DIN0207_L6.3mm_D2.5mm_P7.62mm_Horizontal, symbol Device:R
- added SW1: RotaryEncoder_Switch, Rotary_Encoder:RotaryEncoder_Alps_EC12E-Switch_Vertical_H20mm, symbol Device:RotaryEncoder_Switch
- added U2: 6N138, Package_DIP:DIP-8_W7.62mm_Socket, symbol Isolator:6N138
- added U3: 74HCT125, Package_SO:SOIC-14_3.9x8.7mm_P1.27mm, symbol 74hct125:74HCT125
- U1: renamed from U?; footprint RPi_Pico:RPi_Pico_SMD_TH -> MCU_RaspberryPi_and_Boards:RPi_Pico_TH
Connections:
- net at U1.14 (GPIO10): now also U3.9 (3A)
- net at U1.15 (GPIO11): now also U3.12 (4A)
- net GND: now reaches U1.18 (GND)
- net GND: now also C1.2, C2.1, C3.2, C4.1, J3.2, J4.S, J5.4 (Pin_4), J6.1 (Pin_1), J7.1 (Pin_1), J8.2, SW1.C, SW1.S2, U2.5 (GND), U3.1 (1~{OE}), U3.10 (3~{OE}), U3.13 (4~{OE}), U3.4 (2~{OE}), U3.7 (GND)
- net at U1.2 (GPIO1): now also R1.1, R4.1, U2.6 (VO2)
- net at U1.24 (GPIO18): now also SW1.B
- net at U1.25 (GPIO19): now also SW1.A
- net at U1.26 (GPIO20): now also J5.1 (Pin_1)
- net at U1.27 (GPIO21): now also J5.2 (Pin_2)
- net at U1.29 (GPIO22): now also SW1.S1
- net +3.3V: now reaches U1.36 (3V3)
- net +3.3V: now also C1.1, C2.2, J5.3 (Pin_3), R1.2, R3.2, U2.8 (VCC)
- net +5V: now reaches U1.39 (VSYS)
- net +5V: now also C3.1, C4.2, J6.4 (Pin_4), J7.4 (Pin_4), J9.1 (Pin_1), U3.14 (VCC)
- net at U1.4 (GPIO2): now also U3.2 (1A)
- net at U1.5 (GPIO3): now also U3.5 (2A)
- new net: D1.1 (K), R2.1, U2.2 (C1)
- new net: D1.2 (A), J1.T, J2.5, U2.3 (C2)
- new net: J10.2 (Pin_2), J8.1, J9.2 (Pin_2)
- new net: J10.1 (Pin_1), J8.3
- new net: J3.5, J4.T, R4.2
- new net: J7.2 (Pin_2), U3.8 (3Y)
- new net: J7.3 (Pin_3), U3.11 (4Y)
- new net: J6.2 (Pin_2), U3.3 (1Y)
- new net: J6.3 (Pin_3), U3.6 (2Y)
- new net: J3.4, J4.R, R3.1
- new net: J1.R, J2.4, R2.2
- no-connect marks 0 -> 35
