File: hardware/v1/v1.kicad_pcb (KiCad board)
At the start: 2 copper layers, 77.2 x 91.4 mm, 34 parts, among them J1 MIDI in TRS, J10 Batt, J2 MIDI IN, J3 MIDI THRU, J4 MIDI thru TRS, J5 SSD1306 - I2C, J6 DotStar1/k:GND, J7 DotStar2/k:GND, J8 Barrel_Jack_Switch, J9 On/Off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

Commit message: Putting switch on bottom
Parts:
- J9: moved to B.Cu
Changed lines of the file:
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@@
       ) (layer "F.SilkS") (width 0) (fill solid))
   )
-  (footprint "Connector_JST:JST_XH_B2B-XH-A_1x02_P2.50mm_Vertical" (layer "F.Cu")
-    (at 125.75 119.871)
-    (descr "JST XH series connector, B2B-XH-A (http://www.jst-mfg.com/product/pdf/eng/eXH.pdf), generated with kicad-footprint-generator")
-    (tags "connector JST XH vertical")
-    (property "Sheetfile" "v1.kicad_sch")
-    (property "Sheetname" "")
-    (attr through_hole)
-    (fp_text reference "J9" (at 1.25 -3.55) (layer "F.SilkS")
-      (effects (font (size 1 1) (thickness 0.15)))
-    )
-    (fp_text value "On/Off" (at 1.25 4.6) (layer "F.SilkS")
-      (effects (font (size 1 1) (thickness 0.15)))
-    )
-    (fp_text user "${REFERENCE}" (at 1.25 2.7) (layer "F.Fab")
-      (effects (font (size 1 1) (thickness 0.15)))
-    )
-    (fp_line (start 3.25 -1.7) (end 5.05 -1.7) (layer "F.SilkS") (width 0.12))
-    (fp_line (start 5.05 -2.45) (end 3.25 -2.45) (layer "F.SilkS") (width 0.12))
-    (fp_line (start 1.75 -1.7) (end 1.75 -2.45) (layer "F.SilkS") (width 0.12))
-    (fp_line (start -0.75 -2.45) (end -2.55 -2.45) (layer "F.SilkS") (width 0.12))
-    (fp_line (start 5.05 -0.2) (end 4.3 -0.2) (layer "F.SilkS") (width 0.12))
-    (fp_line (start -2.56 3.51) (end 5.06 3.51) (layer "F.SilkS") (width 0.12))
-    (fp_line (start -1.8 -0.2) (end -1.8 2.75) (layer "F.SilkS") (width 0.12))
-    (fp_line (start 5.05 -1.7) (end 5.05 -2.45) (layer "F.SilkS") (width 0.12))
-    (fp_line (start 5.06 -2.46) (end -2.56 -2.46) (layer "F.SilkS") (width 0.12))
-    (fp_line (start 0.75 -2.45) (end 0.75 -1.7) (layer "F.SilkS") (width 0.12))
-    (fp_line (start -1.6 -2.75) (end -2.85 -2.75) (layer "F.SilkS") (width 0.12))
-    (fp_line (start -0.75 -1.7) (end -0.75 -2.45) (layer "F.SilkS") (width 0.12))
-    (fp_line (start -2.55 -2.45) (end -2.55 -1.7) (layer "F.SilkS") (width 0.12))
-    (fp_line (start -1.8 2.75) (end 1.25 2.75) (layer "F.SilkS") (width 0.12))
-    (fp_line (start 3.25 -2.45) (end 3.25 -1.7) (layer "F.SilkS") (width 0.12))
-    (fp_line (start -2.55 -0.2) (end -1.8 -0.2) (layer "F.SilkS") (width 0.12))
-    (fp_line (start 4.3 -0.2) (end 4.3 2.75) (layer "F.SilkS") (width 0.12))
-    (fp_line (start 1.75 -2.45) (end 0.75 -2.45) (layer "F.SilkS") (width 0.12))
-    (fp_line (start 4.3 2.75) (end 1.25 2.75) (layer "F.SilkS") (width 0.12))
-    (fp_line (start -2.85 -2.75) (end -2.85 -1.5) (layer "F.SilkS") (width 0.12))
-    (fp_line (start 5.06 3.51) (end 5.06 -2.46) (layer "F.SilkS") (width 0.12))
-    (fp_line (start -2.56 -2.46) (end -2.56 3.51) (layer "F.SilkS") (width 0.12))
-    (fp_line (start 0.75 -1.7) (end 1.75 -1.7) (layer "F.SilkS") (width 0.12))
-    (fp_line (start -2.55 -1.7) (end -0.75 -1.7) (layer "F.SilkS") (width 0.12))
-    (fp_line (start -2.95 -2.85) (end -2.95 3.9) (layer "F.CrtYd") (width 0.05))
-    (fp_line (start 5.45 -2.85) (end -2.95 -2.85) (layer "F.CrtYd") (width 0.05))
-    (fp_line (start 5.45 3.9) (end 5.45 -2.85) (layer "F.CrtYd") (width 0.05))
-    (fp_line (start -2.95 3.9) (end 5.45 3.9) (layer "F.CrtYd") (width 0.05))
-    (fp_line (start 0 -1.35) (end 0.625 -2.35) (layer "F.Fab") (width 0.1))
-    (fp_line (start 4.95 3.4) (end 4.95 -2.35) (layer "F.Fab") (width 0.1))
-    (fp_line (start -2.45 -2.35) (end -2.45 3.4) (layer "F.Fab") (width 0.1))
-    (fp_line (start -2.45 3.4) (end 4.95 3.4) (layer "F.Fab") (width 0.1))
-    (fp_line (start -0.625 -2.35) (end 0 -1.35) (layer "F.Fab") (width 0.1))
-    (fp_line (start 4.95 -2.35) (end -2.45 -2.35) (layer "F.Fab") (width 0.1))
-    (pad "1" thru_hole roundrect (at 0 0) (size 1.7 2) (drill 1) (layers *.Cu *.Mask) (roundrect_rratio 0.1470588235)
-      (net 3 "+5V") (pinfunction "Pin_1") (pintype "passive"))
-    (pad "2" thru_hole oval (at 2.5 0) (size 1.7 2) (drill 1) (layers *.Cu *.Mask)
-      (net 21 "Net-(J10-Pad2)") (pinfunction "Pin_2") (pintype "passive"))
-    (model "${KICAD6_3DMODEL_DIR}/Connector_JST.3dshapes/JST_XH_B2B-XH-A_1x02_P2.50mm_Vertical.wrl"
-      (offset (xyz 0 0 0))
-      (scale (xyz 1 1 1))
-      (rotate (xyz 0 0 0))
-    )
-  )
   (footprint "Capacitor_THT:CP_Radial_D7.5mm_P2.50mm" (layer "F.Cu")
     (at 124.6054 109.728 180)
@@
       (net 14 "Net-(J3-Pad5)") (pintype "passive"))
   )
+  (footprint "Connector_JST:JST_XH_B2B-XH-A_1x02_P2.50mm_Vertical" (layer "B.Cu")
+    (at 125.75 119.871)
+    (descr "JST XH series connector, B2B-XH-A (http://www.jst-mfg.com/product/pdf/eng/eXH.pdf), generated with kicad-footprint-generator")
+    (tags "connector JST XH vertical")
+    (property "Sheetfile" "v1.kicad_sch")
+    (property "Sheetname" "")
+    (attr through_hole)
+    (fp_text reference "J9" (at 1.25 3.55) (layer "B.SilkS")
+      (effects (font (size 1 1) (thickness 0.15)) (justify mirror))
+    )
+    (fp_text value "On/Off" (at 1.25 -4.6) (layer "B.SilkS")
+      (effects (font (size 1 1) (thickness 0.15)) (justify mirror))
+    )
+    (fp_text user "${REFERENCE}" (at 1.25 -2.7) (layer "B.Fab")
+      (effects (font (size 1 1) (thickness 0.15)) (justify mirror))
+    )
+    (fp_line (start 3.25 1.7) (end 5.05 1.7) (layer "B.SilkS") (width 0.12))
+    (fp_line (start 5.05 2.45) (end 3.25 2.45) (layer "B.SilkS") (width 0.12))
+    (fp_line (start 1.75 1.7) (end 1.75 2.45) (layer "B.SilkS") (width 0.12))
+    (fp_line (start -0.75 2.45) (end -2.55 2.45) (layer "B.SilkS") (width 0.12))
+    (fp_line (start 5.05 0.2) (end 4.3 0.2) (layer "B.SilkS") (width 0.12))
+    (fp_line (start -2.56 -3.51) (end 5.06 -3.51) (layer "B.SilkS") (width 0.12))
+    (fp_line (start -1.8 0.2) (end -1.8 -2.75) (layer "B.SilkS") (width 0.12))
+    (fp_line (start 5.05 1.7) (end 5.05 2.45) (layer "B.SilkS") (width 0.12))
+    (fp_line (start 5.06 2.46) (end -2.56 2.46) (layer "B.SilkS") (width 0.12))
+    (fp_line (start 0.75 2.45) (end 0.75 1.7) (layer "B.SilkS") (width 0.12))
+    (fp_line (start -1.6 2.75) (end -2.85 2.75) (layer "B.SilkS") (width 0.12))
+    (fp_line (start -0.75 1.7) (end -0.75 2.45) (layer "B.SilkS") (width 0.12))
+    (fp_line (start -2.55 2.45) (end -2.55 1.7) (layer "B.SilkS") (width 0.12))
+    (fp_line (start -1.8 -2.75) (end 1.25 -2.75) (layer "B.SilkS") (width 0.12))
+    (fp_line (start 3.25 2.45) (end 3.25 1.7) (layer "B.SilkS") (width 0.12))
+    (fp_line (start -2.55 0.2) (end -1.8 0.2) (layer "B.SilkS") (width 0.12))
+    (fp_line (start 4.3 0.2) (end 4.3 -2.75) (layer "B.SilkS") (width 0.12))
+    (fp_line (start 1.75 2.45) (end 0.75 2.45) (layer "B.SilkS") (width 0.12))
+    (fp_line (start 4.3 -2.75) (end 1.25 -2.75) (layer "B.SilkS") (width 0.12))
+    (fp_line (start -2.85 2.75) (end -2.85 1.5) (layer "B.SilkS") (width 0.12))
+    (fp_line (start 5.06 -3.51) (end 5.06 2.46) (layer "B.SilkS") (width 0.12))
+    (fp_line (start -2.56 2.46) (end -2.56 -3.51) (layer "B.SilkS") (width 0.12))
+    (fp_line (start 0.75 1.7) (end 1.75 1.7) (layer "B.SilkS") (width 0.12))
+    (fp_line (start -2.55 1.7) (end -0.75 1.7) (layer "B.SilkS") (width 0.12))
+    (fp_line (start -2.95 2.85) (end -2.95 -3.9) (layer "B.CrtYd") (width 0.05))
+    (fp_line (start 5.45 2.85) (end -2.95 2.85) (layer "B.CrtYd") (width 0.05))
+    (fp_line (start 5.45 -3.9) (end 5.45 2.85) (layer "B.CrtYd") (width 0.05))
+    (fp_line (start -2.95 -3.9) (end 5.45 -3.9) (layer "B.CrtYd") (width 0.05))
+    (fp_line (start 0 1.35) (end 0.625 2.35) (layer "B.Fab") (width 0.1))
+    (fp_line (start 4.95 -3.4) (end 4.95 2.35) (layer "B.Fab") (width 0.1))
+    (fp_line (start -2.45 2.35) (end -2.45 -3.4) (layer "B.Fab") (width 0.1))
+    (fp_line (start -2.45 -3.4) (end 4.95 -3.4) (layer "B.Fab") (width 0.1))
+    (fp_line (start -0.625 2.35) (end 0 1.35) (layer "B.Fab") (width 0.1))
+    (fp_line (start 4.95 2.35) (end -2.45 2.35) (layer "B.Fab") (width 0.1))
+    (pad "1" thru_hole roundrect (at 0 0) (size 1.7 2) (drill 1) (layers *.Cu *.Mask) (roundrect_rratio 0.1470588235)
+      (net 3 "+5V") (pinfunction "Pin_1") (pintype "passive"))
+    (pad "2" thru_hole oval (at 2.5 0) (size 1.7 2) (drill 1) (layers *.Cu *.Mask)
+      (net 21 "Net-(J10-Pad2)") (pinfunction "Pin_2") (pintype "passive"))
+    (model "${KICAD6_3DMODEL_DIR}/Connector_JST.3dshapes/JST_XH_B2B-XH-A_1x02_P2.50mm_Vertical.wrl"
+      (offset (xyz 0 0 0))
+      (scale (xyz 1 1 1))
+      (rotate (xyz 0 0 0))
+    )
+  )
   (footprint "Connector_BarrelJack:BarrelJack_CUI_PJ-102AH_Horizontal" (layer "B.Cu")
